Commit message: Robot model loading and pointers

File: ros2_ws/left_resolved.urdf (robot description, URDF)
Before this commit: robot dual, 33 links, 32 joints
Links:
- added link world
Joints:
- added joint left_base_joint: type fixed, parent world, child left_summit_base_footprint, origin xyz=-1.32 0 0.123316 rpy=0 0 0

File: ros2_ws/right_resolved.urdf (robot description, URDF)
Before this commit: robot dual, 33 links, 32 joints
Links:
- added link world
Joints:
- added joint right_base_joint: type fixed, parent world, child right_summit_base_footprint, origin xyz=1.32 0 0.123316 rpy=0 0 0
