Commit message: robot models updated with paletta, paletta model fix

File: ros2_ws/left_resolved_paletta.urdf (robot description, URDF)
Before this commit: robot left_srm, 34 links, 33 joints
Links:
- removed link ur_left_finger_left
- removed link ur_left_finger_right
- removed link ur_left_finger_tip
- removed link ur_left_robotiq_hand
- added link ur_left_paletta; collision mesh filename=file:///ros2_ws/src/simod_proj/paletta_simod/meshes/paletta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; visual mesh filename=file:///ros2_ws/src/simod_proj/paletta_simod/meshes/paletta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
Joints:
- removed joint ur_left_bl_to_leftFinger
- removed joint ur_left_gripper_joint
- removed joint ur_left_leftFinger_to_rightFinger
- removed joint ur_left_rightFinger_to_tip
- added joint ur_left_ee_joint: type fixed, parent ur_left_tool0, child ur_left_paletta, origin xyz=0 0 0 rpy=0 -1.57 0

File: ros2_ws/right_resolved_paletta.urdf (robot description, URDF)
Before this commit: robot right_srm, 34 links, 33 joints
Links:
- removed link ur_right_finger_left
- removed link ur_right_finger_right
- removed link ur_right_finger_tip
- removed link ur_right_robotiq_hand
- added link ur_right_paletta; collision mesh filename=file:///ros2_ws/src/simod_proj/paletta_simod/meshes/paletta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; visual mesh filename=file:///ros2_ws/src/simod_proj/paletta_simod/meshes/paletta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
Joints:
- removed joint ur_right_bl_to_leftFinger
- removed joint ur_right_gripper_joint
- removed joint ur_right_leftFinger_to_rightFinger
- removed joint ur_right_rightFinger_to_tip
- added joint ur_right_ee_joint: type fixed, parent ur_right_tool0, child ur_right_paletta, origin xyz=0 0 0 rpy=0 -1.57 0

File: ros2_ws/src/simod_proj/ur/xacro/srm.urdf.xacro (robot description, xacro)
@@ -15,5 +15,5 @@
     <parent link="world"/>
     <child link="left_summit_base_footprint"/>
-    <origin xyz="-1.32 0 0.123316" rpy="0 0 0"/>
+    <origin xyz="0 0 0.123316" rpy="0 0 0"/>
   </joint>
   <!-- Connect the right robot to the world -->
@@ -21,5 +21,5 @@
     <parent link="world"/>
     <child link="right_summit_base_footprint"/>
-    <origin xyz="1.32 0 0.123316" rpy="0 0 0"/>
+    <origin xyz="0 0 0.123316" rpy="0 0 0"/>
   </joint>
   <!-- istanziare la macro-->
@@ -402,15 +402,10 @@
   </gazebo>
   <!-- *origin-->
-  <link name="ur_left_robotiq_hand">
-    <inertial>
-      <origin rpy="0 0 0" xyz="-0.000186465319378916 -0.0001114030990718 0.0493790267181303"/>
-      <mass value="0.356812979694354"/>
-      <inertia ixx="0.0014834" ixy="-3.7391E-06" ixz="3.3528E-06" iyy="0.002045" iyz="8.3983E-06" izz="0.0020565"/>
-    </inertial>
-    <visual>
-      <origin rpy="0 0 0" xyz="0 0 0"/>
-      <geometry>
-        <mesh filename="file:///ros2_ws/install/robotiq_hand_e/share/robotiq_hand_e/meshes/wiring_gripper.stl">
-                </mesh>
+    <link name="ur_left_paletta">
+    <visual>
+      <origin rpy="0 -1.570796327 3.141592654" xyz="0 0 0"/>
+      <geometry>
+        <mesh filename="file:///ros2_ws/src/simod_proj/paletta_simod/meshes/paletta_v1_simplified_to_mm.stl">
+        </mesh>
       </geometry>
       <material name="">
@@ -421,105 +416,15 @@
       <origin rpy="0 0 0" xyz="0 0 0"/>
       <geometry>
-        <mesh filename="file:///ros2_ws/install/robotiq_hand_e/share/robotiq_hand_e/meshes/wiring_gripper.stl">
-                    </mesh>
+        <mesh filename="file:///ros2_ws/src/simod_proj/paletta_simod/meshes/paletta_v1_simplified_to_mm.stl">
+        </mesh>
       </geometry>
     </collision>
     <gravity>0</gravity>
   </link>
-  <joint name="ur_left_gripper_joint" type="fixed">
-    <!-- <xacro:insert_block name="origin" /> -->
-    <origin rpy="0 -1.57 0" xyz="0 0 0"/>
+  <joint name="ur_left_ee_joint" type="fixed">
     <parent link="ur_left_tool0"/>
-    <child link="ur_left_robotiq_hand"/>
-  </joint>
-  <link name="ur_left_finger_left">
-    <inertial>
-      <origin rpy="0 0 0" xyz="-0.0410573464020155 0.0465900929893167 -0.00138976696740157"/>
-      <mass value="0.0235898515527658"/>
-      <inertia ixx="4.9675E-05" ixy="2.4802E-05" ixz="-4.8356E-07" iyy="2.7862E-05" iyz="2.8798E-06" izz="7.1379E-05"/>
-    </inertial>
-    <visual>
-      <origin rpy="0 0 0" xyz="0 0 0"/>
-      <geometry>
-        <mesh filename="file:///ros2_ws/install/robotiq_hand_e/share/robotiq_hand_e/meshes/hand_e_finger_left_.stl">
-                </mesh>
-      </geometry>
-      <material name="">
-        <color rgba="0.792156862745098 0.819607843137255 0.933333333333333 1"/>
-      </material>
-    </visual>
-    <collision>
-      <origin rpy="0 0 0" xyz="0 0 0"/>
-      <geometry>
-        <mesh filename="file:///ros2_ws/install/robotiq_hand_e/share/robotiq_hand_e/meshes/hand_e_finger_left_.stl">
-                </mesh>
-      </geometry>
-    </collision>
-    <gravity>0</gravity>
-  </link>
-  <joint name="ur_left_bl_to_leftFinger" type="fixed">
-    <origin rpy="0 3.14 -1.57" xyz="0.1133 -0.014 -0.026"/>
-    <parent link="ur_left_robotiq_hand"/>
-    <child link="ur_left_finger_left"/>
-    <axis xyz="0 0 1"/>
-    <limit effort="185" lower="-0.0082" upper="0.0" velocity="150"/>
-  </joint>
-  <link name="ur_left_finger_right">
-    <inertial>
-      <origin rpy="0 0 0" xyz="0.0405573941670405 0.0465900943222486 -0.00138976565433925"/>
-      <mass value="0.0235898505817182"/>
-      <inertia ixx="4.9675E-05" ixy="-2.4835E-05" ixz="4.5546E-07" iyy="2.7862E-05" iyz="2.8798E-06" izz="7.1379E-05"/>
-    </inertial>
-    <visual>
-      <origin rpy="0 0 0" xyz="0 0 0"/>
-      <geometry>
-        <mesh filename="file:///ros2_ws/install/robotiq_hand_e/share/robotiq_hand_e/meshes/hand_e_finger_right_.stl">
-                </mesh>
-      </geometry>
-      <material name="">
-        <color rgba="0.792156862745098 0.819607843137255 0.933333333333333 1"/>
-      </material>
-    </visual>
-    <collision>
-      <origin rpy="0 0 0" xyz="0 0 0"/>
-      <geometry>
-        <mesh filename="file:///ros2_ws/install/robotiq_hand_e/share/robotiq_hand_e/meshes/hand_e_finger_right_.stl">
-                </mesh>
-      </geometry>
-    </collision>
-    <gravity>0</gravity>
-  </link>
-  <joint name="ur_left_leftFinger_to_rightFinger" type="fixed">
-    <origin rpy="0 0 0" xyz="0.0285 0 -0.052"/>
-    <parent link="ur_left_finger_left"/>
-    <child link="ur_left_finger_right"/>
-    <axis xyz="0 0 1"/>
-    <limit effort="185" lower="0.0" upper="0.045" velocity="150"/>
-  </joint>
-  <link name="ur_left_finger_tip"/>
-  <joint name="ur_left_rightFinger_to_tip" type="fixed">
-    <origin rpy="1.5707963267948966 0 1.5707963267948966" xyz="0.157 0 0.0018"/>
-    <parent link="ur_left_robotiq_hand"/>
-    <child link="ur_left_finger_tip"/>
-    <dynamics damping="0" friction="0"/>
-  </joint>
-  <transmission name="ur_left_leftFinger_trans">
-    <type>transmission_interface/SimpleTransmission</type>
-    <joint name="ur_left_bl_to_leftFinger">
-      <hardwareInterface>hardware_interface/PositionJointInterface</hardwareInterface>
-    </joint>
-    <actuator name="ur_left_leftFinger_motor">
-      <mechanicalReduction>1</mechanicalReduction>
-    </actuator>
-  </transmission>
-  <transmission name="ur_left_rightFinger_trans">
-    <type>transmission_interface/SimpleTransmission</type>
-    <joint name="ur_left_leftFinger_to_rightFinger">
-      <hardwareInterface>hardware_interface/PositionJointInterface</hardwareInterface>
-    </joint>
-    <actuator name="ur_left_rightFinger_motor">
-      <mechanicalReduction>1</mechanicalReduction>
-    </actuator>
-  </transmission>
+    <child link="ur_left_paletta"/>
+    <origin rpy="0 -1.57 0" xyz="0 0 0"/> <!-- Set the correct pose here -->
+  </joint>
   <!-- ***************** -->
   <!-- Imported elements -->
@@ -1183,7 +1088,4 @@
     <plugin filename="libgazebo_ros2_control.so" name="left_gazebo_ros2_control">
       <parameters>/ros2_ws/install/ur/share/ur/config/left_controller.yaml</parameters>
-      <ros>
-        <namespace>left</namespace>
-      </ros>
     </plugin>
   </gazebo>
@@ -1573,124 +1475,29 @@
     </gazebo>
     <!-- *origin-->
-    <link name="ur_right_robotiq_hand">
-    <inertial>
-        <origin rpy="0 0 0" xyz="-0.000186465319378916 -0.0001114030990718 0.0493790267181303"/>
-        <mass value="0.356812979694354"/>
-        <inertia ixx="0.0014834" ixy="-3.7391E-06" ixz="3.3528E-06" iyy="0.002045" iyz="8.3983E-06" izz="0.0020565"/>
-    </inertial>
-    <visual>
-        <origin rpy="0 0 0" xyz="0 0 0"/>
-        <geometry>
-        <mesh filename="file:///ros2_ws/install/robotiq_hand_e/share/robotiq_hand_e/meshes/wiring_gripper.stl">
-                </mesh>
-        </geometry>
-        <material name="">
+        <link name="ur_right_paletta">
+    <visual>
+      <origin rpy="0 -1.570796327 3.141592654" xyz="0 0 0"/>
+      <geometry>
+        <mesh filename="file:///ros2_ws/src/simod_proj/paletta_simod/meshes/paletta_v1_simplified_to_mm.stl">
+        </mesh>
+      </geometry>
+      <material name="">
         <color rgba="0.792156862745098 0.819607843137255 0.933333333333333 1"/>
-        </material>
-    </visual>
-    <collision>
-        <origin rpy="0 0 0" xyz="0 0 0"/>
-        <geometry>
-        <mesh filename="file:///ros2_ws/install/robotiq_hand_e/share/robotiq_hand_e/meshes/wiring_gripper.stl">
-                    </mesh>
-        </geometry>
+      </material>
+    </visual>
+    <collision>
+      <origin rpy="0 0 0" xyz="0 0 0"/>
+      <geometry>
+        <mesh filename="file:///ros2_ws/src/simod_proj/paletta_simod/meshes/paletta_v1_simplified_to_mm.stl">
+        </mesh>
+      </geometry>
     </collision>
     <gravity>0</gravity>
-    </link>
-    <joint name="ur_right_gripper_joint" type="fixed">
-    <!-- <xacro:insert_block name="origin" /> -->
-    <origin rpy="0 -1.57 0" xyz="0 0 0"/>
+  </link>
+  <joint name="ur_right_ee_joint" type="fixed">
     <parent link="ur_right_tool0"/>
-    <child link="ur_right_robotiq_hand"/>
-    </joint>
-    <link name="ur_right_finger_left">
-    <inertial>
-        <origin rpy="0 0 0" xyz="-0.0410573464020155 0.0465900929893167 -0.00138976696740157"/>
-        <mass value="0.0235898515527658"/>
-        <inertia ixx="4.9675E-05" ixy="2.4802E-05" ixz="-4.8356E-07" iyy="2.7862E-05" iyz="2.8798E-06" izz="7.1379E-05"/>
-    </inertial>
-    <visual>
-        <origin rpy="0 0 0" xyz="0 0 0"/>
-        <geometry>
-        <mesh filename="file:///ros2_ws/install/robotiq_hand_e/share/robotiq_hand_e/meshes/hand_e_finger_left_.stl">
-                </mesh>
-        </geometry>
-        <material name="">
-        <color rgba="0.792156862745098 0.819607843137255 0.933333333333333 1"/>
-        </material>
-    </visual>
-    <collision>
-        <origin rpy="0 0 0" xyz="0 0 0"/>
-        <geometry>
-        <mesh filename="file:///ros2_ws/install/robotiq_hand_e/share/robotiq_hand_e/meshes/hand_e_finger_left_.stl">
-                </mesh>
-        </geometry>
-    </collision>
-    <gravity>0</gravity>
-    </link>
-    <joint name="ur_right_bl_to_leftFinger" type="fixed">
-    <origin rpy="0 3.14 -1.57" xyz="0.1133 -0.014 -0.026"/>
-    <parent link="ur_right_robotiq_hand"/>
-    <child link="ur_right_finger_left"/>
-    <axis xyz="0 0 1"/>
-    <limit effort="185" lower="-0.0082" upper="0.0" velocity="150"/>
-    </joint>
-    <link name="ur_right_finger_right">
-    <inertial>
-        <origin rpy="0 0 0" xyz="0.0405573941670405 0.0465900943222486 -0.00138976565433925"/>
-        <mass value="0.0235898505817182"/>
-        <inertia ixx="4.9675E-05" ixy="-2.4835E-05" ixz="4.5546E-07" iyy="2.7862E-05" iyz="2.8798E-06" izz="7.1379E-05"/>
-    </inertial>
-    <visual>
-        <origin rpy="0 0 0" xyz="0 0 0"/>
-        <geometry>
-        <mesh filename="file:///ros2_ws/install/robotiq_hand_e/share/robotiq_hand_e/meshes/hand_e_finger_right_.stl">
-                </mesh>
-        </geometry>
-        <material name="">
-        <color rgba="0.792156862745098 0.819607843137255 0.933333333333333 1"/>
-        </material>
-    </visual>
-    <collision>
-        <origin rpy="0 0 0" xyz="0 0 0"/>
-        <geometry>
-        <mesh filename="file:///ros2_ws/install/robotiq_hand_e/share/robotiq_hand_e/meshes/hand_e_finger_right_.stl">
-                </mesh>
-        </geometry>
-    </collision>
-    <gravity>0</gravity>
-    </link>
-    <joint name="ur_right_leftFinger_to_rightFinger" type="fixed">
-    <origin rpy="0 0 0" xyz="0.0285 0 -0.052"/>
-    <parent link="ur_right_finger_left"/>
-    <child link="ur_right_finger_right"/>
-    <axis xyz="0 0 1"/>
-    <limit effort="185" lower="0.0" upper="0.045" velocity="150"/>
-    </joint>
-    <link name="ur_right_finger_tip"/>
-    <joint name="ur_right_rightFinger_to_tip" type="fixed">
-    <origin rpy="1.5707963267948966 0 1.5707963267948966" xyz="0.174 0 0.0018"/>
-    <parent link="ur_right_robotiq_hand"/>
-    <child link="ur_right_finger_tip"/>
-    <dynamics damping="0" friction="0"/>
-    </joint>
-    <transmission name="ur_right_leftFinger_trans">
-    <type>transmission_interface/SimpleTransmission</type>
-    <joint name="ur_right_bl_to_leftFinger">
-        <hardwareInterface>hardware_interface/PositionJointInterface</hardwareInterface>
-    </joint>
-    <actuator name="ur_right_leftFinger_motor">
-        <mechanicalReduction>1</mechanicalReduction>
-    </actuator>
-    </transmission>
-    <transmission name="ur_right_rightFinger_trans">
-    <type>transmission_interface/SimpleTransmission</type>
-    <joint name="ur_right_leftFinger_to_rightFinger">
-        <hardwareInterface>hardware_interface/PositionJointInterface</hardwareInterface>
-    </joint>
-    <actuator name="ur_right_rightFinger_motor">
-        <mechanicalReduction>1</mechanicalReduction>
-    </actuator>
-    </transmission>
+    <child link="ur_right_paletta"/>
+    <origin rpy="0 -1.57 0" xyz="0 0 0"/> <!-- Set the correct pose here -->
+  </joint>
     <!-- ***************** -->
     <!-- Imported elements -->

Commit message: MOVEIT-GAZEBO SYNC FIX

File: ros2_ws/left_resolved_paletta.urdf (robot description, URDF)
Before this commit: robot left_srm, 31 links, 30 joints
Joints:
- joint left_base_joint: origin xyz=-1.32 0 0.123316 rpy=0 0 0 -> xyz=0 0 0.123316 rpy=0 0 0

File: ros2_ws/right_resolved_paletta.urdf (robot description, URDF)
Before this commit: robot right_srm, 31 links, 30 joints
Joints:
- joint right_base_joint: origin xyz=1.32 0 0.123316 rpy=0 0 0 -> xyz=0 0 0.123316 rpy=0 0 0

File: ros2_ws/src/simod_proj/ur/xacro/srm.urdf.xacro (robot description, xacro)
@@ -402,5 +402,5 @@
   </gazebo>
   <!-- *origin-->
-    <link name="ur_left_paletta">
+  <link name="ur_left_paletta">
     <visual>
       <origin rpy="0 -1.570796327 3.141592654" xyz="0 0 0"/>
@@ -1077,6 +1077,6 @@
       <odometryRate>50.0</odometryRate>
       <robot_base_frame>left_summit_base_footprint</robot_base_frame>
-      <publish_odom>true</publish_odom>
-      <publish_odom_tf>true</publish_odom_tf>
+      <publish_odom>false</publish_odom>
+      <publish_odom_tf>false</publish_odom_tf>
       <enableYAxis>true</enableYAxis>
     </plugin>
@@ -2150,6 +2150,6 @@
         <odometryRate>50.0</odometryRate>
         <robot_base_frame>right_summit_base_footprint</robot_base_frame>
-        <publish_odom>true</publish_odom>
-        <publish_odom_tf>true</publish_odom_tf>
+        <publish_odom>false</publish_odom>
+        <publish_odom_tf>false</publish_odom_tf>
         <enableYAxis>true</enableYAxis>
     </plugin>

File: ros2_ws/src/simod_proj/ur/xacro/ur_spawn.urdf.xacro (robot description, xacro)
@@ -2,6 +2,4 @@
 <robot xmlns:xacro="http://wiki.ros.org/xacro" name="dual">
     <xacro:include filename="$(find ur_description)/urdf/ur_macro.xacro"/>
-    <xacro:include filename="$(find robotiq_hand_e)/urdf/robotiq_wiring.urdf.xacro"/>
-    <xacro:include filename="$(find robotiq_hand_e)/urdf/robotiq_trasmission.xacro"/>
     <xacro:arg name="connected_to" default=""/>
     <xacro:arg name="namespace" default=""/>
@@ -102,6 +100,30 @@
         <origin xyz="$(arg xyz)" rpy="$(arg rpy_base_ur)"/>
     </xacro:ur_robot>
-    <xacro:wiring_gripper prefix="$(arg tf_prefix)" parent="$(arg parent_hand)" rpy="$(arg rpy)" finger_tip_cor="$(arg finger_tip_cor)"/>
-    <xacro:robotiq_trasmission prefix="$(arg tf_prefix)" hw_interface="$(arg hardware_interface)"/>
+    <xacro:wiring_gripper prefix="$(arg tf_prefix)" parent="$(arg parent_hand)" rpy="$(arg rpy)"/>
+    <link name="ur_left_paletta">
+        <visual>
+        <origin rpy="0 -1.570796327 3.141592654" xyz="0 0 0"/>
+        <geometry>
+            <mesh filename="file:///ros2_ws/src/simod_proj/paletta_simod/meshes/paletta_v1_simplified_to_mm.stl">
+            </mesh>
+        </geometry>
+        <material name="">
+            <color rgba="0.792156862745098 0.819607843137255 0.933333333333333 1"/>
+        </material>
+        </visual>
+        <collision>
+        <origin rpy="0 0 0" xyz="0 0 0"/>
+        <geometry>
+            <mesh filename="file:///ros2_ws/src/simod_proj/paletta_simod/meshes/paletta_v1_simplified_to_mm.stl">
+            </mesh>
+        </geometry>
+        </collision>
+        <gravity>0</gravity>
+    </link>
+    <joint name="ur_$(arg namespace)_paletta_joint" type="fixed">
+        <parent link="$(arg parent_hand)"/>
+        <child link="ur_$(arg namespace)_paletta"/>
+        <origin xyz="0.157 0 0.0018" rpy="0 0 0"/>
+    </joint>
     <xacro:if value="$(arg spawn_gazebo_base)">
         <xacro:include filename="$(find base)/xacro/base_spawn.urdf.xacro"/>

File: ros2_ws/src/summit_xl_common/summit_xl_description/urdf/bases/summit_xl_base.gazebo.xacro (robot description, xacro)
@@ -44,5 +44,5 @@
 	      <robot_base_frame>${prefix}_base_footprint</robot_base_frame>
 		  <publish_odom>true</publish_odom>
-      	  <publish_odom_tf>true</publish_odom_tf>
+      	  <publish_odom_tf>false</publish_odom_tf>
 		  <enableYAxis>true</enableYAxis>
 	    </plugin>

Commit message: odometry fix

File: ros2_ws/left_resolved_paletta.urdf (robot description, URDF)
Before this commit: robot left_srm, 31 links, 30 joints
Links:
- removed link world
Joints:
- removed joint left_base_joint

File: ros2_ws/right_resolved_paletta.urdf (robot description, URDF)
Before this commit: robot right_srm, 31 links, 30 joints
Links:
- removed link world
Joints:
- removed joint right_base_joint

File: ros2_ws/src/simod_proj/ur/xacro/srm.urdf.xacro (robot description, xacro)
@@ -15,5 +15,5 @@
     <parent link="world"/>
     <child link="left_summit_base_footprint"/>
-    <origin xyz="0 0 0" rpy="0 0 0"/>
+    <origin xyz="0 0 0.123316" rpy="0 0 0"/>
   </joint>
   <!-- Connect the right robot to the world -->
@@ -21,5 +21,5 @@
     <parent link="world"/>
     <child link="right_summit_base_footprint"/>
-    <origin xyz="0 0 0" rpy="0 0 0"/>
+    <origin xyz="0 0 0.123316" rpy="0 0 0"/>
   </joint>
   <!-- istanziare la macro-->

Commit message: demo pick and place (case 1) completo

File: ros2_ws/left_resolved_paletta.urdf (robot description, URDF)
Before this commit: robot left_srm, 30 links, 29 joints
Links:
- link ur_left_forearm_link: geometry visual mesh filename=file:///ros2_ws/install/ur_description/share/ur_description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
- link ur_left_paletta: geometry visual mesh filename=file:///ros2_ws/src/simod_proj/paletta_simod/meshes/paletta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
- link ur_left_upper_arm_link: geometry visual mesh filename=file:///ros2_ws/install/ur_description/share/ur_description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
- link ur_left_wrist_1_link: geometry visual mesh filename=file:///ros2_ws/install/ur_description/share/ur_description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
- link ur_left_wrist_2_link: geometry visual mesh filename=file:///ros2_ws/install/ur_description/share/ur_description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
- link ur_left_wrist_3_link: geometry visual mesh filename=file:///ros2_ws/install/ur_description/share/ur_description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

File: ros2_ws/right_resolved_paletta.urdf (robot description, URDF)
Before this commit: robot right_srm, 30 links, 29 joints
Links:
- link ur_right_forearm_link: geometry visual mesh filename=file:///ros2_ws/install/ur_description/share/ur_description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
- link ur_right_paletta: geometry visual mesh filename=file:///ros2_ws/src/simod_proj/paletta_simod/meshes/paletta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
- link ur_right_shoulder_link: geometry visual mesh filename=file:///ros2_ws/install/ur_description/share/ur_description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
- link ur_right_upper_arm_link: geometry visual mesh filename=file:///ros2_ws/install/ur_description/share/ur_description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
- link ur_right_wrist_1_link: geometry visual mesh filename=file:///ros2_ws/install/ur_description/share/ur_description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
- link ur_right_wrist_2_link: geometry visual mesh filename=file:///ros2_ws/install/ur_description/share/ur_description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
- link ur_right_wrist_3_link: geometry visual mesh filename=file:///ros2_ws/install/ur_description/share/ur_description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

Commit message: camera update, bt approach delay, single launch restruct

File: ros2_ws/left_resolved_paletta.urdf (robot description, URDF)
Before this commit: robot left_srm, 30 links, 29 joints
Links:
- added link ur_left_camera_link; visual box size=0.010 0.03 0.03
- added link ur_left_camera_link_optical
- added link ur_left_camera_mount_link, mass 0.01; visual box size=0.009 0.06 0.06
Joints:
- added joint ur_left_camera_joint: type fixed, parent ur_left_camera_mount_link, child ur_left_camera_link, origin xyz=0 0 0 rpy=0 0 0
- added joint ur_left_camera_optical_joint: type fixed, parent ur_left_camera_link, child ur_left_camera_link_optical, origin xyz=0 0 0 rpy=0 0 0
- added joint ur_left_wrist_1_camera_mount_joint: type revolute, parent ur_left_wrist_1_link, child ur_left_camera_mount_link, origin xyz=0 -0.09 -0.18 rpy=-1.57 0 -1.57, axis 0 1 0, limit lower=-1.57 upper=1.57 effort=0.5 velocity=1

File: ros2_ws/right_resolved_paletta.urdf (robot description, URDF)
Before this commit: robot right_srm, 30 links, 29 joints
Links:
- added link ur_right_camera_link; visual box size=0.010 0.03 0.03
- added link ur_right_camera_link_optical
- added link ur_right_camera_mount_link, mass 0.01; visual box size=0.009 0.06 0.06
Joints:
- added joint ur_right_camera_joint: type fixed, parent ur_right_camera_mount_link, child ur_right_camera_link, origin xyz=0 0 0 rpy=0 0 0
- added joint ur_right_camera_optical_joint: type fixed, parent ur_right_camera_link, child ur_right_camera_link_optical, origin xyz=0 0 0 rpy=0 0 0
- added joint ur_right_wrist_1_camera_mount_joint: type revolute, parent ur_right_wrist_1_link, child ur_right_camera_mount_link, origin xyz=0 -0.09 -0.18 rpy=-1.57 0 -1.57, axis 0 1 0, limit lower=-1.57 upper=1.57 effort=0.5 velocity=1
