Commit message: approach demo completed

File: ros2_ws/left_resolved_paletta.urdf (robot description, URDF)
Before this commit: robot left_srm, 33 links, 32 joints
Joints:
- joint ur_left_camera_joint: origin xyz=0 0 0 rpy=0 0 0 -> xyz=0 0 0 rpy=-1.57 0 0
- joint ur_left_wrist_1_camera_mount_joint: axis 0 1 0 -> (none); limit lower=-1.57 upper=1.57 effort=0.5 velocity=1 -> (none); origin xyz=0 -0.09 -0.18 rpy=-1.57 0 -1.57 -> xyz=0 -0.09 -0.18 rpy=0 0 -1.57; type revolute -> fixed

File: ros2_ws/right_resolved_paletta.urdf (robot description, URDF)
Before this commit: robot right_srm, 33 links, 32 joints
Joints:
- joint ur_right_camera_joint: origin xyz=0 0 0 rpy=0 0 0 -> xyz=0 0 0 rpy=1.57 0 0
- joint ur_right_wrist_1_camera_mount_joint: axis 0 1 0 -> (none); limit lower=-1.57 upper=1.57 effort=0.5 velocity=1 -> (none); origin xyz=0 -0.09 -0.18 rpy=-1.57 0 -1.57 -> xyz=0 -0.09 -0.18 rpy=0 0 -1.57; type revolute -> fixed

Commit message: Demo completa integrata TP

File: ros2_ws/left_resolved_paletta.urdf (robot description, URDF)
Before this commit: robot left_srm, 33 links, 32 joints
Joints:
- joint ur_left_wrist_1_camera_mount_joint: origin xyz=0 -0.09 -0.18 rpy=0 0 -1.57 -> xyz=0 -0.09 -0.18 rpy=0 0 -1.77

File: ros2_ws/right_resolved_paletta.urdf (robot description, URDF)
Before this commit: robot right_srm, 33 links, 32 joints
Joints:
- joint ur_right_camera_joint: origin xyz=0 0 0 rpy=1.57 0 0 -> xyz=0 0 0 rpy=1.57 0 0.20
