Commit message: Planning scene update

File: ros2_ws/src/simod_proj/ur/xacro/srm.urdf.xacro (robot description, xacro)
@@ -12,14 +12,14 @@
   <link name="world"/>
   <!-- Connect the left robot to the world -->
-  <joint name="left_base_joint" type="fixed">
+  <joint name="left_base_joint" type="floating">
     <parent link="world"/>
     <child link="left_summit_base_footprint"/>
-    <origin xyz="-0.66 0 0" rpy="0 0 0"/> <!-- Adjust position as needed -->
+    <origin xyz="-1.32 0 0.123316" rpy="0 0 0"/> <!-- Adjust position as needed -->
   </joint>
   <!-- Connect the right robot to the world -->
-  <joint name="right_base_joint" type="fixed">
+  <joint name="right_base_joint" type="floating">
     <parent link="world"/>
     <child link="right_summit_base_footprint"/>
-    <origin xyz="0.66 0 0" rpy="0 0 0"/> <!-- Adjust position as needed -->
+    <origin xyz="1.32 0 0.123316" rpy="0 0 0"/> <!-- Adjust position as needed -->
   </joint>
   <!-- istanziare la macro-->

Commit message: Scene sync rviz

File: ros2_ws/src/simod_proj/ur/xacro/srm.urdf.xacro (robot description, xacro)
@@ -12,14 +12,14 @@
   <link name="world"/>
   <!-- Connect the left robot to the world -->
-  <joint name="left_base_joint" type="floating">
+  <joint name="left_base_joint" type="fixed">
     <parent link="world"/>
     <child link="left_summit_base_footprint"/>
-    <origin xyz="-1.32 0 0.123316" rpy="0 0 0"/> <!-- Adjust position as needed -->
+    <origin xyz="-1.32 0 0.123316" rpy="0 0 0"/>
   </joint>
   <!-- Connect the right robot to the world -->
-  <joint name="right_base_joint" type="floating">
+  <joint name="right_base_joint" type="fixed">
     <parent link="world"/>
     <child link="right_summit_base_footprint"/>
-    <origin xyz="1.32 0 0.123316" rpy="0 0 0"/> <!-- Adjust position as needed -->
+    <origin xyz="1.32 0 0.123316" rpy="0 0 0"/>
   </joint>
   <!-- istanziare la macro-->

Commit message: preliminary mtc task, updated gazebo_sync to broadcast tf.

File: ros2_ws/src/simod_proj/ur/xacro/srm.urdf.xacro (robot description, xacro)
@@ -12,5 +12,5 @@
   <link name="world"/>
   <!-- Connect the left robot to the world -->
-  <joint name="left_base_joint" type="fixed">
+  <joint name="left_base_joint" type="planar">
     <parent link="world"/>
     <child link="left_summit_base_footprint"/>
@@ -18,5 +18,5 @@
   </joint>
   <!-- Connect the right robot to the world -->
-  <joint name="right_base_joint" type="fixed">
+  <joint name="right_base_joint" type="planar">
     <parent link="world"/>
     <child link="right_summit_base_footprint"/>

Commit message: z axis offset fix

File: ros2_ws/src/simod_proj/ur/xacro/srm.urdf.xacro (robot description, xacro)
@@ -15,5 +15,5 @@
     <parent link="world"/>
     <child link="left_summit_base_footprint"/>
-    <origin xyz="0 0 0.123316" rpy="0 0 0"/>
+    <origin xyz="0 0 0" rpy="0 0 0"/>
   </joint>
   <!-- Connect the right robot to the world -->
@@ -21,5 +21,5 @@
     <parent link="world"/>
     <child link="right_summit_base_footprint"/>
-    <origin xyz="0 0 0.123316" rpy="0 0 0"/>
+    <origin xyz="0 0 0" rpy="0 0 0"/>
   </joint>
   <!-- istanziare la macro-->

Commit message: semantic error fixes, mtc planning scene update, logs

File: ros2_ws/src/simod_proj/ur/xacro/srm.urdf.xacro (robot description, xacro)
@@ -1475,5 +1475,5 @@
     </gazebo>
     <!-- *origin-->
-        <link name="ur_right_paletta">
+  <link name="ur_right_paletta">
     <visual>
       <origin rpy="0 -1.570796327 3.141592654" xyz="0 0 0"/>

Commit message: restructored launch, simple controller manager mod, action controller skeleton

File: ros2_ws/src/simod_proj/ur/xacro/srm.urdf.xacro (robot description, xacro)
@@ -1083,5 +1083,5 @@
   </gazebo>
   <!-- <xacro:summit_xl prefix="${prefix)}" publish_bf="true" hq="true"/> -->
-  <gazebo reference="world">
+  <!-- <gazebo reference="world">
         </gazebo>
   <gazebo>
@@ -1095,5 +1095,5 @@
     </ros>
     <update_rate>1.0</update_rate>
-  </plugin>
+  </plugin> -->
   <!-- ROBOT RIGHT: istanziare la macro-->
   <ros2_control name="right_ur" type="system">
@@ -2158,5 +2158,5 @@
     <gazebo reference="world">
         </gazebo>
-    <gazebo>
+    <!-- <gazebo>
     <plugin filename="libgazebo_ros2_control.so" name="right_gazebo_ros2_control">
         <parameters>/ros2_ws/install/ur/share/ur/config/right_controller.yaml</parameters>
@@ -2165,10 +2165,10 @@
         </ros>
     </plugin>
-    </gazebo>
-    <plugin filename="libgazebo_ros2_state.so" name="right_gazebo_ros_state">
+    </gazebo> -->
+    <!-- <plugin filename="libgazebo_ros2_state.so" name="right_gazebo_ros_state">
     <ros>
         <namespace>right</namespace>
     </ros>
     <update_rate>1.0</update_rate>
-    </plugin>
+    </plugin> -->
 </robot>

File: ros2_ws/src/srm_simod_moveit_config/config/srm.ros2_control.xacro (robot description, xacro)
@@ -8,33 +8,9 @@
                 <plugin>mock_components/GenericSystem</plugin>
             </hardware>
-            <joint name="right_summit_back_left_wheel_joint">
+            <joint name="right_base_joint">
                 <command_interface name="position"/>
                 <command_interface name="velocity"/>
                 <state_interface name="position">
-                  <param name="initial_value">${initial_positions['right_summit_back_left_wheel_joint']}</param>
-                </state_interface>
-                <state_interface name="velocity"/>
-            </joint>
-            <joint name="right_summit_back_right_wheel_joint">
-                <command_interface name="position"/>
-                <command_interface name="velocity"/>
-                <state_interface name="position">
-                  <param name="initial_value">${initial_positions['right_summit_back_right_wheel_joint']}</param>
-                </state_interface>
-                <state_interface name="velocity"/>
-            </joint>
-            <joint name="right_summit_front_left_wheel_joint">
-                <command_interface name="position"/>
-                <command_interface name="velocity"/>
-                <state_interface name="position">
-                  <param name="initial_value">${initial_positions['right_summit_front_left_wheel_joint']}</param>
-                </state_interface>
-                <state_interface name="velocity"/>
-            </joint>
-            <joint name="right_summit_front_right_wheel_joint">
-                <command_interface name="position"/>
-                <command_interface name="velocity"/>
-                <state_interface name="position">
-                  <param name="initial_value">${initial_positions['right_summit_front_right_wheel_joint']}</param>
+                  <param name="initial_value">${initial_positions['right_base_joint']}</param>
                 </state_interface>
                 <state_interface name="velocity"/>
@@ -88,33 +64,9 @@
                 <state_interface name="velocity"/>
             </joint>
-            <joint name="left_summit_back_left_wheel_joint">
+            <joint name="left_base_joint">
                 <command_interface name="position"/>
                 <command_interface name="velocity"/>
                 <state_interface name="position">
-                  <param name="initial_value">${initial_positions['left_summit_back_left_wheel_joint']}</param>
-                </state_interface>
-                <state_interface name="velocity"/>
-            </joint>
-            <joint name="left_summit_back_right_wheel_joint">
-                <command_interface name="position"/>
-                <command_interface name="velocity"/>
-                <state_interface name="position">
-                  <param name="initial_value">${initial_positions['left_summit_back_right_wheel_joint']}</param>
-                </state_interface>
-                <state_interface name="velocity"/>
-            </joint>
-            <joint name="left_summit_front_left_wheel_joint">
-                <command_interface name="position"/>
-                <command_interface name="velocity"/>
-                <state_interface name="position">
-                  <param name="initial_value">${initial_positions['left_summit_front_left_wheel_joint']}</param>
-                </state_interface>
-                <state_interface name="velocity"/>
-            </joint>
-            <joint name="left_summit_front_right_wheel_joint">
-                <command_interface name="position"/>
-                <command_interface name="velocity"/>
-                <state_interface name="position">
-                  <param name="initial_value">${initial_positions['left_summit_front_right_wheel_joint']}</param>
+                  <param name="initial_value">${initial_positions['left_base_joint']}</param>
                 </state_interface>
                 <state_interface name="velocity"/>
