Commit message: updates, BT, etc.

File: ros2_ws/src/simod_proj/ur/xacro/left_resolved_paletta.urdf (robot description, URDF)
Before this commit: robot srm_left, 30 links, 29 joints
Joints:
- added joint left_base_joint: type planar, parent world, child left_summit_base_footprint, origin xyz=0 0 0 rpy=0 0 0

Commit message: usecase update

File: ros2_ws/src/simod_proj/ur/xacro/left_resolved_paletta.urdf (robot description, URDF)
Before this commit: robot srm_left, 30 links, 30 joints
Joints:
- removed joint left_base_joint
